File: RPi_TPU_DevBoard/RPi_TPU_DevBoard.kicad_sch (KiCad schematic)
At the start: 1 part

Commit message: Initial commit copy from my gitlab repository
Parts:
- removed U?: G313-06329-00, MODULE_G313-06329-00, symbol G313-06329-00:G313-06329-00
Other:
- added sheet CM4_GPIO (CM4_GPIO.kicad_sch)
- added sheet CM4_High_Speed_Buses (CM4_High_Speed_Buses.kicad_sch)
- added sheet Google TPU (Google_TPU.kicad_sch)
- added sheet USB HUB (usb.kicad_sch)
